Commit message: resources: bring Fetch meshes under resources/fetch/ + add holonomic base inertials
Copied 53 Fetch meshes (~19 MB: .dae visual, .stl collision) from
thirdparty/vamp_preview/resources/fetch/meshes/ into
resources/fetch/meshes/ so resources/fetch/fetch.urdf's
`package://meshes/*` references resolve without requiring the vamp
submodule. This is the canonical spot — the URDF was already there,
the meshes just weren't.

Added minimal <inertial> blocks (mass=0.001 kg, diagonal I=1e-6) to
x_link / y_link / theta_link — the three holonomic-base
intermediate links that previously had only a placeholder comment.
MuJoCo-based validators (used under the hood by Genesis's URDF
parser) reject moving bodies with zero mass; Sapien/ManiSkill and
VAMP already tolerated the missing inertials, so this change is a
no-op for existing backends.

Pre-commit: bumped check-added-large-files from 2 MB to 5 MB so
the two biggest Fetch meshes (base_link.dae 4.6 MB, torso_lift_link.dae
3.3 MB) can land. Still keeps the guardrail against accidental
multi-MB binaries but accommodates standard robotics art.

Verified: `import genesis; scene.add_entity(gs.morphs.URDF(...));
scene.build()` now succeeds. 12 joints / 17 DOF / 12 links —
matches expected Fetch structure (root + x/y/theta holonomic base +
torso + 7 arm + head pan/tilt + gripper).

Unblocks Step 12 (Genesis backend) which needs a loadable Fetch
URDF to implement GenesisFetchSimBackend.

File: resources/fetch/fetch.urdf (robot description, URDF)
Before this commit: robot fetch, 21 links, 20 joints
Links:
- link theta_link: mass None -> 0.001
- link x_link: mass None -> 0.001
- link y_link: mass None -> 0.001
